Commit message: feat(mesh): OBJ with Chinese mtllib -> binary STL, full-shell URDF
Foxglove does not read .mtl and lists OBJ as its weakest format; the
Menagerie OBJs reference a missing `mtllib 深色橡胶.001.mtl`, so every
<mesh> failed and the 3D panel showed TF arrows only.

- scripts/convert_meshes.py (trimesh, pypi): 16x .obj -> binary .stl,
  28MB -> 8.7MB, face counts identical, bounds diff <=1.1e-8 m
- urdf/go2.urdf: all 30 mesh refs .stl via package:// (kept, no HTTP);
  added missing base_3/base_4 shell + _1 cover plates on every leg link
  (was 19 refs/9 files, now 30/16); joint order matches sim_node
- validated: URDF parses (13 links/12 joints, no broken refs), live
  /tf carries world->base, world->base_gt + all 12 leg frames @458Hz,
  /robot_description serves STL URDF, bridge :8765 advertises all,
  16 STLs where package:// resolves; fusion still tracking
- trimesh added as pypi dep (assimp conda pkg has no CLI)
- foxglove/go2_demo.json: URDF layer Source=Topic /robot_description,
  meshUpAxis=z_up (STL has no orientation; Foxglove defaults y-up),
  marked STARTER until overwritten by Studio export
- README Demo section: ./scripts/go2_demo.sh flow + video/GIF player
  notes (GitHub strips <video>; use CDN bare URL or GIF via
  scripts/make_gif.sh); go2_http.urdf kept in sync as fallback,
  HTTP :8000 server stays in launch until package:// confirmed in Studio

Co-authored-by: mesh-stl

File: ros2/otolith_description/urdf/go2.urdf (robot description, URDF)
Before this commit: robot go2, 13 links, 12 joints
Links:
- link FL_calf: geometry visual mesh filename=package://otolith_description/meshes/calf_0.stl; visual mesh filename=package://otolith_description/meshes/calf_1.stl
- link FL_hip: geometry visual mesh filename=package://otolith_description/meshes/hip_0.stl; visual mesh filename=package://otolith_description/meshes/hip_1.stl
- link FL_thigh: geometry visual mesh filename=package://otolith_description/meshes/thigh_0.stl; visual mesh filename=package://otolith_description/meshes/thigh_1.stl
- link FR_calf: geometry visual mesh filename=package://otolith_description/meshes/calf_mirror_0.stl; visual mesh filename=package://otolith_description/meshes/calf_mirror_1.stl
- link FR_hip: geometry visual mesh filename=package://otolith_description/meshes/hip_0.stl; visual mesh filename=package://otolith_description/meshes/hip_1.stl
- link FR_thigh: geometry visual mesh filename=package://otolith_description/meshes/thigh_mirror_0.stl; visual mesh filename=package://otolith_description/meshes/thigh_mirror_1.stl
- link RL_calf: geometry visual mesh filename=package://otolith_description/meshes/calf_0.stl; visual mesh filename=package://otolith_description/meshes/calf_1.stl
- link RL_hip: geometry visual mesh filename=package://otolith_description/meshes/hip_0.stl; visual mesh filename=package://otolith_description/meshes/hip_1.stl
- link RL_thigh: geometry visual mesh filename=package://otolith_description/meshes/thigh_0.stl; visual mesh filename=package://otolith_description/meshes/thigh_1.stl
- link RR_calf: geometry visual mesh filename=package://otolith_description/meshes/calf_mirror_0.stl; visual mesh filename=package://otolith_description/meshes/calf_mirror_1.stl
- link RR_hip: geometry visual mesh filename=package://otolith_description/meshes/hip_0.stl; visual mesh filename=package://otolith_description/meshes/hip_1.stl
- link RR_thigh: geometry visual mesh filename=package://otolith_description/meshes/thigh_mirror_0.stl; visual mesh filename=package://otolith_description/meshes/thigh_mirror_1.stl
- link base: geometry collision box size=0.35 0.14 0.07; visual mesh filename=package://otolith_description/meshes/base_0.stl scale=1 1 1

File: ros2/otolith_description/urdf/go2_http.urdf (robot description, URDF)
Before this commit: robot go2, 13 links, 12 joints
Links:
- link FL_calf: geometry visual mesh filename=http://localhost:8000/calf_0.stl; visual mesh filename=http://localhost:8000/calf_1.stl
- link FL_hip: geometry visual mesh filename=http://localhost:8000/hip_0.stl; visual mesh filename=http://localhost:8000/hip_1.stl
- link FL_thigh: geometry visual mesh filename=http://localhost:8000/thigh_0.stl; visual mesh filename=http://localhost:8000/thigh_1.stl
- link FR_calf: geometry visual mesh filename=http://localhost:8000/calf_mirror_0.stl; visual mesh filename=http://localhost:8000/calf_mirror_1.stl
- link FR_hip: geometry visual mesh filename=http://localhost:8000/hip_0.stl; visual mesh filename=http://localhost:8000/hip_1.stl
- link FR_thigh: geometry visual mesh filename=http://localhost:8000/thigh_mirror_0.stl; visual mesh filename=http://localhost:8000/thigh_mirror_1.stl
- link RL_calf: geometry visual mesh filename=http://localhost:8000/calf_0.stl; visual mesh filename=http://localhost:8000/calf_1.stl
- link RL_hip: geometry visual mesh filename=http://localhost:8000/hip_0.stl; visual mesh filename=http://localhost:8000/hip_1.stl
- link RL_thigh: geometry visual mesh filename=http://localhost:8000/thigh_0.stl; visual mesh filename=http://localhost:8000/thigh_1.stl
- link RR_calf: geometry visual mesh filename=http://localhost:8000/calf_mirror_0.stl; visual mesh filename=http://localhost:8000/calf_mirror_1.stl
- link RR_hip: geometry visual mesh filename=http://localhost:8000/hip_0.stl; visual mesh filename=http://localhost:8000/hip_1.stl
- link RR_thigh: geometry visual mesh filename=http://localhost:8000/thigh_mirror_0.stl; visual mesh filename=http://localhost:8000/thigh_mirror_1.stl
- link base: geometry collision box size=0.35 0.14 0.07; visual mesh filename=http://localhost:8000/base_0.stl scale=1 1 1
